Commit message: Tiny bug fix

File: urdf/my_robot.xacro (robot description, xacro)
@@ -121,5 +121,7 @@
 		<visual name='camera_visual'>
 			<origin xyz="0 0 0" rpy="0 0 0"/>
-			<box size="0.05 0.05 0.05"/>
+			<geometry>
+				<box size="0.05 0.05 0.05"/>
+			</geometry>
 		</visual>
 		<collision name='camera_collision'>

Commit message: Added RTAB mapping launch file

File: urdf/my_robot.xacro (robot description, xacro)
@@ -174,3 +174,10 @@
 		<child link='hokuyo'/>
 	</joint>
+	<joint name="camera_optical_joint" type="fixed">
+    <origin xyz="0 0 0" rpy="-1.5707 0 -1.5707"/>
+    <parent link="camera"/>
+    <child link="camera_link_optical"/>
+  	</joint>
+  	<link name="camera_link_optical">
+  	</link>
 </robot>
